File: PCB/bm_controller.sch (KiCad schematic (older format))
At the start: 27 parts, among them J1 Conn_01x08, J2 Conn_01x03, Q1 BSC040N10NS5, U1 ESP32-DOIT-EVALKIT, U2 IRS2890DS, U3 LM5017MR, U4 LMT87DCK

Commit message: added gitignore, advanced with schematic design
Parts:
- added J1: Conn_01x02, symbol Connector_Generic:Conn_01x02
- added Q? (x5): BSC040N10NS5, Package_TO_SOT_SMD:TDSON-8-1, symbol Transistor_FET:CSD19534Q5A
- added U? (x2): IRS2890DS, Package_SO:SOIC-14_3.9x8.7mm_P1.27mm, symbol IRS2890DS:IRS2890DS
- renumbered C7 to C5, C5 to C6, C6 to C7, J1 to J2, J2 to J3, R6 to R4, R7 to R5, R4 to R6, R5 to R7, U3 to U1, U4 to U2, U1 to U3, U2 to U4
Connections:
- net labels added: COM, M1, M2, M3, REF
- wire segments 83 -> 167
Other:
- moved on the sheet: Q1
